Commit message: Restore control GUI and fix serial, ARM and emote reliability
The 204 KB control GUI had been overwritten by a 24 KB stub that also
dropped the MOTION-ownership and ARM controls, so the robot could not be
driven at all. It was never committed, so it was rebuilt by replaying the
233 apply_patch operations from the editor transcripts and reconciling the
result against the surviving bytecode until all 174 code objects compiled
identically.

Serial path: the link ran at 57600 with servo updates gated on an idle
wire, so a 28% duty cycle starved the 20 ms interpolation tick, and a
corrupted frame failed to feed the 750 ms watchdog while its own error
reply lengthened the next loop block and corrupted the next frame. Baud is
now 250000 (exact from 16 MHz, 0.0% error), the servo tick only defers for
a partially received line, and rejectFrame() separates "the host is still
talking" from "we have no usable target" so isolated corruption reports
instead of silently disarming. The NeoPixel blackout is now covered by a
measured inter-frame window rather than by running the wire slowly.

ARM stopped disarming at random: any focus change while armed dropped both
layers to HOLD. Losing focus now zeroes the inputs immediately and starts a
20 s grace period, so an abandoned console still ends safe while a glance
at another window does not. MOTION ownership is also re-asserted at 5 Hz
because the router aged it off the pose stream and let it lapse whenever a
gait stopped.

Emote range was bounded by four separate ceilings. Limits are now set from
sweeps of the controller's own IK preflight rather than by guesswork:
amplitude 2.0x (wave/heart bind at 2.3x because they lift a foot) and
push-up depth 3.0x for 60 mm of travel. The emote body-height floor is
split from the standing envelope, since a planted-foot emote folds the leg
rather than reaching with it; standing, walking and manual pose are
unchanged.

GUI status labels now reserve a fixed number of text lines, so a longer
message no longer reflows the layout and resizes the window under the
operator's cursor.

Firmware verified with arduino --verify; suite is 472 passing. Contract
tests were re-pointed at the new behaviour rather than relaxed.

Co-Authored-By: Claude Opus 5 (1M context) <noreply@anthropic.com>

File: src/volt_description/urdf/ros2_control.xacro (robot description, xacro)
@@ -96,5 +96,5 @@
           <parameters>$(find volt_description)/config/controllers.yaml</parameters>
           <controller_manager_name>controller_manager</controller_manager_name>
-          <position_proportional_gain>0.35</position_proportional_gain>
+          <position_proportional_gain>0.1</position_proportional_gain>
         </plugin>
       </gazebo>

File: src/volt_description/urdf/volt.urdf.xacro (robot description, xacro)
@@ -4,4 +4,5 @@
 <xacro:include filename="$(find volt_description)/urdf/gazebo.xacro"/>
 <xacro:arg name="sim_backend" default="gz"/>
+<xacro:arg name="actuator_profile" default="simulation"/>
   <material name="yellow">
     <color rgba="0.92 0.83 0.0 1"/>
@@ -14,4 +15,15 @@
   </material>
   <!-- Params -->
+  <!-- Keep the proven simulation profile as default.  The opt-in hardware
+       profile matches the production firmware's 120 deg/s channel slew and
+       uses a less idealized effort/damping envelope without changing ROS/IK
+       joint limits or physical calibration. -->
+  <xacro:property name="hardware_actuators" value="${'$(arg actuator_profile)' == 'td8130mg'}"/>
+  <xacro:property name="shoulder_velocity" value="${2.0}"/>
+  <xacro:property name="leg_velocity" value="${2.0944 if hardware_actuators else 3.0}"/>
+  <xacro:property name="foot_velocity" value="${2.0944 if hardware_actuators else 4.5}"/>
+  <xacro:property name="joint_effort" value="${6.0 if hardware_actuators else 20.0}"/>
+  <xacro:property name="joint_damping" value="${0.9 if hardware_actuators else 0.6}"/>
+  <xacro:property name="joint_friction" value="${0.15 if hardware_actuators else 0.1}"/>
   <xacro:property name="body_length" value="0.140" />
   <xacro:property name="body_width" value="0.110" />
@@ -68,6 +80,6 @@
       <axis xyz="1 0 0"/>
       <origin rpy="0 0 0" xyz="${shiftx} ${shifty} 0"/>
-      <limit effort="20.0" lower="-0.548" upper="0.548" velocity="2.0"/>
-      <dynamics damping="0.6" friction="0.1"/>
+      <limit effort="${joint_effort}" lower="-0.548" upper="0.548" velocity="${shoulder_velocity}"/>
+      <dynamics damping="${joint_damping}" friction="${joint_friction}"/>
     </joint>
   </xacro:macro>
@@ -129,6 +141,6 @@
       <axis xyz="0 1 0"/>
       <origin rpy="0 0 0" xyz="0 ${shift} 0"/>
-      <limit effort="20.0" lower="-2.666" upper="1.548" velocity="3.0"/>
-      <dynamics damping="0.6" friction="0.1"/>
+      <limit effort="${joint_effort}" lower="-2.666" upper="1.548" velocity="${leg_velocity}"/>
+      <dynamics damping="${joint_damping}" friction="${joint_friction}"/>
     </joint>
     <joint name="${pos}_leg_cover_joint" type="fixed">
@@ -173,6 +185,6 @@
       <axis xyz="0 1 0"/>
       <origin rpy="0 0 0" xyz="0 0 -${leg_length}"/>
-      <limit effort="20.0" lower="-2.6" upper="0.1" velocity="4.5"/>
-      <dynamics damping="0.6" friction="0.1"/>
+      <limit effort="${joint_effort}" lower="-2.6" upper="0.1" velocity="${foot_velocity}"/>
+      <dynamics damping="${joint_damping}" friction="${joint_friction}"/>
     </joint>
   </xacro:macro>

Commit message: Rebuild walking ground-up: two servo-budgeted gaits verified in Ignition
The nine previous gaits across four code paths are removed and replaced by
one engine with exactly two gaits: a two-beat diagonal trot (duty 0.58,
1.1 s cycle, 0.12 m/s) and a four-beat lateral-sequence amble (duty 0.76,
2.0 s cycle, three feet always planted, body sway away from the swinging
side). Every historical gait name aliases onto one of the two, so saved
profiles and old commands keep working.

The core design change is that the TD-8130MG's behavior under load is now a
configuration contract instead of an afterthought. The swing leg is
unloaded and can run near the servo's ~375 deg/s free speed; the stance
legs carry the body but rotate slowly. Loading a gait config sweeps a full
cycle at its maximum command through the real IK and refuses any
configuration exceeding 80 deg/s on loaded stance joints, 190 deg/s on the
unloaded swing leg (firmware ceiling 240), or 6500 deg/s^2 of commanded
acceleration. A config that loads is a config the servos can execute, so
the downstream velocity/acceleration limiters are fault ceilings rather
than trajectory shapers. Real-robot profiles re-run the same sweep when
applied and cannot smuggle in an infeasible gait.

Stance feet are world-locked (zero skate by construction), swing transfer
uses smoothstep with a sin^2 lift, and touchdown targets are frozen
world-frame points, so command changes never jerk an airborne foot. A
forced stop latches: a held joystick cannot restart motion until the
controller observes a truly neutral command and releases the latch (the
release path exists because an idle engine never sees the neutral itself).

Gazebo Ignition now models the servo under load: the td8130mg profile
carries the 240 deg/s firmware velocity ceiling and a derated 2.8 N.m
stall-torque effort limit, and the gz_ros2_control tracking gain rises
from 0.1 to 18.0 so the effort clamp, not a soft gain, is what slows a
loaded joint. Verified headless across six cases (trot forward/turn/
lateral/max, amble forward/turn): zero falls, trot 76% velocity
realization at 0.10 m/s with roll p95 4 deg, amble stable at 2-3 deg.
The same verification exposed and fixed the old stack's real disease:
an 18 rad/s^2 acceleration clamp against ~85 rad/s^2 of gait demand had
been shredding trajectories (20% realization, 13 deg rocking).

Control rate drops to 100 Hz everywhere; the Python controller measured
94 Hz against the old 200 Hz timer with 12k missed deadlines, and the
engine is dt-based so the rate is a sampling choice. Removed: the three
fast-trot tools, physical_fast_trot.yaml, FAST_TROT.md, five test files,
the GUI fast-trot tuning panel, /volt/fast_trot_tuning, the standalone
forward-walk firmware sketch, and all launch arguments that carried them.
Docs rewritten to match. Suite: 415 passing.

Co-Authored-By: Claude Fable 5 <noreply@anthropic.com>

File: src/volt_description/urdf/ros2_control.xacro (robot description, xacro)
@@ -96,5 +96,5 @@
           <parameters>$(find volt_description)/config/controllers.yaml</parameters>
           <controller_manager_name>controller_manager</controller_manager_name>
-          <position_proportional_gain>0.1</position_proportional_gain>
+          <position_proportional_gain>18.0</position_proportional_gain>
         </plugin>
       </gazebo>

File: src/volt_description/urdf/volt.urdf.xacro (robot description, xacro)
@@ -15,15 +15,20 @@
   </material>
   <!-- Params -->
-  <!-- Keep the proven simulation profile as default.  The opt-in hardware
-       profile matches the production firmware's 120 deg/s channel slew and
-       uses a less idealized effort/damping envelope without changing ROS/IK
-       joint limits or physical calibration. -->
+  <!-- Keep the proven simulation profile as default.  The opt-in td8130mg
+       profile models the physical servo under load: velocity capped at the
+       firmware's 240 deg/s slew ceiling (4.1888 rad/s; the servo free speed
+       is ~375 deg/s so firmware is the binding limit), effort capped at a
+       derated 2.8 N.m stall torque (TD-8130MG ~30 kg.cm at 6 V).  With the
+       stiffer tracking gain in ros2_control.xacro the effort clamp - not an
+       artificially soft gain - becomes what slows a loaded joint, so Gazebo
+       reproduces load-dependent tracking lag.  ROS/IK joint limits and
+       physical calibration are unchanged. -->
   <xacro:property name="hardware_actuators" value="${'$(arg actuator_profile)' == 'td8130mg'}"/>
-  <xacro:property name="shoulder_velocity" value="${2.0}"/>
-  <xacro:property name="leg_velocity" value="${2.0944 if hardware_actuators else 3.0}"/>
-  <xacro:property name="foot_velocity" value="${2.0944 if hardware_actuators else 4.5}"/>
-  <xacro:property name="joint_effort" value="${6.0 if hardware_actuators else 20.0}"/>
-  <xacro:property name="joint_damping" value="${0.9 if hardware_actuators else 0.6}"/>
-  <xacro:property name="joint_friction" value="${0.15 if hardware_actuators else 0.1}"/>
+  <xacro:property name="shoulder_velocity" value="${4.1888 if hardware_actuators else 2.0}"/>
+  <xacro:property name="leg_velocity" value="${4.1888 if hardware_actuators else 3.0}"/>
+  <xacro:property name="foot_velocity" value="${4.1888 if hardware_actuators else 4.5}"/>
+  <xacro:property name="joint_effort" value="${2.8 if hardware_actuators else 20.0}"/>
+  <xacro:property name="joint_damping" value="${0.35 if hardware_actuators else 0.6}"/>
+  <xacro:property name="joint_friction" value="${0.10 if hardware_actuators else 0.1}"/>
   <xacro:property name="body_length" value="0.140" />
   <xacro:property name="body_width" value="0.110" />
